File: PCB/kicad/hat/hat.kicad_sch (KiCad schematic)
At the start: 136 parts, among them J1 12V IN, J10 RS485 A B G, J11 12V OUT, J12 HB FLT GND, J2 spare gpio, J3 pH board, J4 EC board, J5 DS18B20, J6 sht31 module, J7 veml7700 module, J8 scd40 module, J9 oled ssd1306, Q1 AOD4184A, Q10 2N7002, Q2 2N7002, Q3 AOD4184A, Q4 AOD4184A, Q5 2N7002, Q6 AO3401A, Q7 2N7002, Q8 AO3401A, Q9 2N7002, U1 LM74700-Q1, U10 ADS1115 module, U11 DS3231MZ, U12 ADM2483BRWZ, U13 B0505S-1WR3, U2 INA226, U3 TPS565208, U4 MCP73831T-2ACI, U5 XL6009E1, U6 LM74700-Q1, U7 LM74700-Q1, U8 AMS1117-3.3, U9 24LC32A

Commit message: i redid everything for one board, one pi 5, and cut some features
Parts:
- removed BT1: 18650 protected, Battery:BatteryHolder_Keystone_1042_1x18650, symbol Device:Battery_Cell
- removed BT2: CR1220, Battery:BatteryHolder_Keystone_3000_1x12mm, symbol Device:Battery_Cell
- removed BZ1: active 5V, Buzzer_Beeper:Buzzer_12x9.5RM7.6, symbol Device:Buzzer
- removed C10, C14, C15, C20, C23, C8, C9: 22u 10V, Capacitor_SMD:C_1206_3216Metric, symbol Device:C
- removed C11, C21, C24, C25, C26, C28, C29, C32, C33, C34, C7: 100n, Capacitor_SMD:C_0805_2012Metric, symbol Device:C
- removed C12, C13, C35, C36: 4u7, Capacitor_SMD:C_0805_2012Metric, symbol Device:C
- removed C16: 220u 10V, Capacitor_THT:CP_Radial_D8.0mm_P3.50mm, symbol Device:C_Polarized
- removed C17, C18: 1u, Capacitor_SMD:C_0805_2012Metric, symbol Device:C
- removed C19: 470u 10V, Capacitor_THT:CP_Radial_D8.0mm_P3.50mm, symbol Device:C_Polarized
- removed C22, C27, C30, C31: 10u, Capacitor_SMD:C_1206_3216Metric, symbol Device:C
- removed C4: 470u 25V, Capacitor_THT:CP_Radial_D10.0mm_P5.00mm, symbol Device:C_Polarized
- removed C5, C6: 10u 25V, Capacitor_SMD:C_1206_3216Metric, symbol Device:C
- removed D1: SMBJ15A, Diode_SMD:D_SMB, symbol Device:D_TVS
- removed D2: charging, LED_SMD:LED_0805_2012Metric, symbol Device:LED
- removed D3: SS34, Diode_SMD:D_SMA, symbol Diode:SS34
- removed D4, D5, D6: SMF5.0A, Diode_SMD:D_SOD-123F, symbol Diode:PESD5V0L1UL
- removed D7: SS14, Diode_SMD:D_SMA, symbol Diode:SS14
- removed D8, D9: SMAJ6.5CA, Diode_SMD:D_SMA, symbol Device:D_TVS
- removed F2, F3: 3A, Fuse:Fuse_1206_3216Metric, symbol Device:Fuse
- removed F4: 7.5A blade, Fuse:FuseHolder_Blade_ATO_Littelfuse_FLR_178.6165, symbol Device:Fuse
- removed H1, H2, H3, H4, H5, H6: M2.5, MountingHole:MountingHole_2.7mm_M2.5, symbol Mechanical:MountingHole
- removed J12: HB FLT GND, Connector_JST:JST_XH_B3B-XH-A_1x03_P2.50mm_Vertical, symbol Connector_Generic:Conn_01x03
- removed J2: spare gpio, Connector_PinHeader_2.54mm:PinHeader_1x04_P2.54mm_Vertical, symbol Connector_Generic:Conn_01x04
- removed J3: pH board, revd:Gravity_TB3, symbol revd:Gravity_Probe
- removed J4: EC board, revd:Gravity_TB3, symbol revd:Gravity_Probe
- removed J5: DS18B20, TerminalBlock_CUI:TerminalBlock_CUI_TB007-508-03_1x03_P5.08mm_Horizontal, symbol Connector:Screw_Terminal_01x03
- removed J7: veml7700 module, Connector_PinHeader_2.54mm:PinHeader_1x04_P2.54mm_Vertical, symbol Connector_Generic:Conn_01x04
- removed J8: scd40 module, Connector_PinHeader_2.54mm:PinHeader_1x04_P2.54mm_Vertical, symbol Connector_Generic:Conn_01x04
- removed J9: oled ssd1306, Connector_PinHeader_2.54mm:PinHeader_1x04_P2.54mm_Vertical, symbol Connector_Generic:Conn_01x04
- removed JP2: term, Jumper:SolderJumper-2_P1.3mm_Open_Pad1.0x1.5mm, symbol Jumper:SolderJumper_2_Open
- removed J_PI: Pi 40 pin, Connector_PinSocket_2.54mm:PinSocket_2x20_P2.54mm_Vertical, symbol Connector_Generic:Conn_02x20_Odd_Even
- removed L1: 4.7u 6A, Inductor_SMD:L_Bourns_SRP7028A_7.3x6.6mm, symbol Device:L
- removed L2: 22u 4A, Inductor_SMD:L_Bourns_SRP7028A_7.3x6.6mm, symbol Device:L
- removed Q1, Q3, Q4: AOD4184A, Package_TO_SOT_SMD:TO-252-2, symbol Transistor_FET:Q_NMOS_GDS
- removed Q10, Q2, Q5, Q7, Q9: 2N7002, Package_TO_SOT_SMD:SOT-23, symbol Transistor_FET:2N7002
- removed Q6, Q8: AO3401A, Package_TO_SOT_SMD:SOT-23, symbol Transistor_FET:AO3401A
- removed R30: 120R, Resistor_SMD:R_0805_2012Metric, symbol Device:R
- removed R31, R32: 47k, Resistor_SMD:R_0805_2012Metric, symbol Device:R
- removed R33: 10k, Resistor_SMD:R_0805_2012Metric, symbol Device:R
- removed R34: 100R, Resistor_SMD:R_0805_2012Metric, symbol Device:R
- removed R_SENSE1, R_SENSE2: 10R, Resistor_SMD:R_0805_2012Metric, symbol Device:R
- removed R_SHUNT: 5m 2512, Resistor_SMD:R_2512_6332Metric_Pad1.40x3.35mm_HandSolder, symbol Device:R
- removed TP1: AIN3, TestPoint:TestPoint_Pad_D1.5mm, symbol Connector:TestPoint
- removed U1, U6, U7: LM74700-Q1, Package_TO_SOT_SMD:SOT-23-6, symbol Power_Management:LM74700
- removed U10: ADS1115 module, revd:ADS1115_Module, symbol Analog_ADC:ADS1115IDGS
- removed U11: DS3231MZ, Package_SO:SOIC-8_3.9x4.9mm_P1.27mm, symbol Timer_RTC:DS3231MZ
- removed U12: ADM2483BRWZ, Package_SO:SOIC-16W_7.5x10.3mm_P1.27mm, symbol Interface_UART:ADM2483xRW
- removed U13: B0505S-1WR3, revd:B0505S_SIP4, symbol revd:B0505S
- removed U2: INA226, Package_SO:MSOP-10_3x3mm_P0.5mm, symbol Sensor_Energy:INA226
- removed U3: TPS565208, Package_TO_SOT_SMD:SOT-23-6, symbol Regulator_Switching:TPS565208
- removed U4: MCP73831T-2ACI, Package_TO_SOT_SMD:SOT-23-5, symbol Battery_Management:MCP73831-2-OT
- removed U5: XL6009E1, revd:TO-263-5_TabNC, symbol revd:XL6009
- removed U8: AMS1117-3.3, Package_TO_SOT_SMD:SOT-223-3_TabPin2, symbol Regulator_Linear:AMS1117-3.3
- removed U9: 24LC32A, Package_SO:SOIC-8_3.9x4.9mm_P1.27mm, symbol Memory_EEPROM:24LC32
- added D1: 1.5KE15A, Diode_THT:D_DO-201AE_P15.24mm_Horizontal, symbol Diode:1.5KExxA
- added D10: pump, LED_THT:LED_D3.0mm, symbol Device:LED
- added D2: SB5H100, Diode_THT:D_DO-201AD_P15.24mm_Horizontal, symbol Diode:SB5H100
- added D3, D4, D5, D8: 1N5819, Diode_THT:D_DO-41_SOD81_P10.16mm_Horizontal, symbol Diode:1N5819
- added D6: 1N5822, Diode_THT:D_DO-201AD_P15.24mm_Horizontal, symbol Diode:1N5822
- added D7: 1N4148, Diode_THT:D_DO-35_SOD27_P7.62mm_Horizontal, symbol Diode:1N4148
- added D9: rail, LED_THT:LED_D3.0mm, symbol Device:LED
- added J12: pump 2, TerminalBlock_CUI:TerminalBlock_CUI_TB007-508-02_1x02_P5.08mm_Horizontal, symbol Connector:Screw_Terminal_01x02
- added J13: pump 3, TerminalBlock_CUI:TerminalBlock_CUI_TB007-508-02_1x02_P5.08mm_Horizontal, symbol Connector:Screw_Terminal_01x02
- added J14: led strip, TerminalBlock_CUI:TerminalBlock_CUI_TB007-508-02_1x02_P5.08mm_Horizontal, symbol Connector:Screw_Terminal_01x02
- added J15: fan, TerminalBlock_CUI:TerminalBlock_CUI_TB007-508-02_1x02_P5.08mm_Horizontal, symbol Connector:Screw_Terminal_01x02
- added J16: flow sensor, TerminalBlock_CUI:TerminalBlock_CUI_TB007-508-03_1x03_P5.08mm_Horizontal, symbol Connector:Screw_Terminal_01x03
- added J2: spare gpio, Connector_PinHeader_2.54mm:PinHeader_1x02_P2.54mm_Vertical, symbol Connector_Generic:Conn_01x02
- added J3: sht31 module, Connector_PinHeader_2.54mm:PinHeader_1x04_P2.54mm_Vertical, symbol Connector_Generic:Conn_01x04
- added J4: veml7700 module, Connector_PinHeader_2.54mm:PinHeader_1x04_P2.54mm_Vertical, symbol Connector_Generic:Conn_01x04
- added J5: scd40 module, Connector_PinHeader_2.54mm:PinHeader_1x04_P2.54mm_Vertical, symbol Connector_Generic:Conn_01x04
- added J7: JSN-SR04T (uart mode), TerminalBlock_CUI:TerminalBlock_CUI_TB007-508-04_1x04_P5.08mm_Horizontal, symbol Connector:Screw_Terminal_01x04
- added J8: pH board, revd:Gravity_TB3, symbol revd:Gravity_Probe
- added J9: EC board, revd:Gravity_TB3, symbol revd:Gravity_Probe
- added J_PI1: Pi 5, 40 pin (tall stacking header), Connector_PinSocket_2.54mm:PinSocket_2x20_P2.54mm_Vertical, symbol Connector_Generic:Conn_02x20_Odd_Even
- added MTG1, MTG2, MTG3, MTG4, MTG5, MTG6: MountingHole, MountingHole:MountingHole_2.7mm_M2.5, symbol Mechanical:MountingHole
- added Q1, Q10: 2N7000, Package_TO_SOT_THT:TO-92_Inline, symbol Transistor_FET:2N7000
- added Q2: IRF9540N, Package_TO_SOT_THT:TO-220-3_Vertical, symbol Transistor_FET:IRF9540N
- added Q3, Q4: BS250, Package_TO_SOT_THT:TO-92_Inline, symbol Transistor_FET:BS250
- added Q5, Q6, Q7, Q8, Q9: IRLZ44N, Package_TO_SOT_THT:TO-220-3_Vertical, symbol Transistor_FET:IRLZ44N
- added R_SHUNT1: 5m, Resistor_THT:R_Axial_DIN0411_L9.9mm_D3.6mm_P15.24mm_Horizontal, symbol Device:R
- added U1: INA226 module 0x40, Connector_PinHeader_2.54mm:PinHeader_1x06_P2.54mm_Vertical, symbol Connector_Generic:Conn_01x06
- added U10: PCA9685 module (i2c), Connector_PinHeader_2.54mm:PinHeader_1x04_P2.54mm_Vertical, symbol Connector_Generic:Conn_01x04
- added U11: PCA9685 ch0 (pump1 pwm), Connector_PinHeader_2.54mm:PinHeader_1x01_P2.54mm_Vertical, symbol Connector_Generic:Conn_01x01
- added U12: PCA9685 ch1 (pump2 pwm), Connector_PinHeader_2.54mm:PinHeader_1x01_P2.54mm_Vertical, symbol Connector_Generic:Conn_01x01
- added U13: PCA9685 ch2 (pump3 pwm), Connector_PinHeader_2.54mm:PinHeader_1x01_P2.54mm_Vertical, symbol Connector_Generic:Conn_01x01
- added U14: PCA9685 ch3 (led pwm), Connector_PinHeader_2.54mm:PinHeader_1x01_P2.54mm_Vertical, symbol Connector_Generic:Conn_01x01
- added U15: PCA9685 ch4 (fan pwm), Connector_PinHeader_2.54mm:PinHeader_1x01_P2.54mm_Vertical, symbol Connector_Generic:Conn_01x01
- added U16: PCA9685 ch5 (rail status led), Connector_PinHeader_2.54mm:PinHeader_1x01_P2.54mm_Vertical, symbol Connector_Generic:Conn_01x01
- added U17: PCA9685 ch6 (pump status led), Connector_PinHeader_2.54mm:PinHeader_1x01_P2.54mm_Vertical, symbol Connector_Generic:Conn_01x01
- added U18: DS3231 RTC module, Connector_PinHeader_2.54mm:PinHeader_1x04_P2.54mm_Vertical, symbol Connector_Generic:Conn_01x04
- added U19: CD40106, Package_DIP:DIP-14_W7.62mm, symbol 4xxx:40106
- added U2: buck module 12V->5V, Connector_PinHeader_2.54mm:PinHeader_1x04_P2.54mm_Vertical, symbol Connector_Generic:Conn_01x04
- added U20: 5V active, Buzzer_Beeper:Buzzer_12x9.5RM7.6, symbol Device:Buzzer
- added U3: AMS1117 3.3V module, Connector_PinHeader_2.54mm:PinHeader_1x03_P2.54mm_Vertical, symbol Connector_Generic:Conn_01x03
- added U4: CD4538, Package_DIP:DIP-16_W7.62mm, symbol 4xxx:4538
- added U5: CD4081, Package_DIP:DIP-14_W7.62mm, symbol 4xxx:4081
- added U6: 24LC32A/P, Package_DIP:DIP-8_W7.62mm, symbol Memory_EEPROM:24LC32
- added U7: ADS1115 module 0x48 (ph/ec + pump3 diff), Connector_PinHeader_2.54mm:PinHeader_1x09_P2.54mm_Vertical, symbol Connector_Generic:Conn_01x09
- added U8: ADS1115 module 0x49 (pump1/pump2 diff), Connector_PinHeader_2.54mm:PinHeader_1x09_P2.54mm_Vertical, symbol Connector_Generic:Conn_01x09
- added U9: ADS1115 module 0x4A (led diff), Connector_PinHeader_2.54mm:PinHeader_1x09_P2.54mm_Vertical, symbol Connector_Generic:Conn_01x09
- C1: value 1u 50V -> 100n; footprint Capacitor_SMD:C_0805_2012Metric -> Capacitor_THT:C_Disc_D3.0mm_W2.0mm_P2.50mm
- C2: value 100n -> 10u 10V; footprint Capacitor_SMD:C_0805_2012Metric -> Capacitor_THT:C_Disc_D3.0mm_W2.0mm_P2.50mm
- C3: footprint Capacitor_SMD:C_0805_2012Metric -> Capacitor_THT:C_Disc_D3.0mm_W2.0mm_P2.50mm
- F1: value 10A blade -> 10A
- J10: value RS485 A B G -> DS18B20
- J11: value 12V OUT -> pump 1
- J6: value sht31 module -> oled ssd1306
- JP1: footprint Jumper:SolderJumper-2_P1.3mm_Open_Pad1.0x1.5mm -> (none)
- R1: value 56k2 -> 470k; footprint Resistor_SMD:R_0805_2012Metric -> Resistor_THT:R_Axial_DIN0207_L6.3mm_D2.5mm_P10.16mm_Horizontal
- R10: value 100k -> 4k7; footprint Resistor_SMD:R_0805_2012Metric -> Resistor_THT:R_Axial_DIN0207_L6.3mm_D2.5mm_P10.16mm_Horizontal
- R11, R14: value 100k -> 100R; footprint Resistor_SMD:R_0805_2012Metric -> Resistor_THT:R_Axial_DIN0207_L6.3mm_D2.5mm_P10.16mm_Horizontal
- R12, R21, R24, R3, R9: value 100k -> 10k; footprint Resistor_SMD:R_0805_2012Metric -> Resistor_THT:R_Axial_DIN0207_L6.3mm_D2.5mm_P10.16mm_Horizontal
- R13: value 100k -> 0.1; footprint Resistor_SMD:R_0805_2012Metric -> Resistor_THT:R_Axial_DIN0411_L9.9mm_D3.6mm_P15.24mm_Horizontal
- R15, R28, R7: footprint Resistor_SMD:R_0805_2012Metric -> Resistor_THT:R_Axial_DIN0207_L6.3mm_D2.5mm_P10.16mm_Horizontal
- R16, R19: value 10k -> 0.1; footprint Resistor_SMD:R_0805_2012Metric -> Resistor_THT:R_Axial_DIN0411_L9.9mm_D3.6mm_P15.24mm_Horizontal
- R17, R20, R23: value 1k -> 100R; footprint Resistor_SMD:R_0805_2012Metric -> Resistor_THT:R_Axial_DIN0207_L6.3mm_D2.5mm_P10.16mm_Horizontal
- R18, R5: value 1k -> 10k; footprint Resistor_SMD:R_0805_2012Metric -> Resistor_THT:R_Axial_DIN0207_L6.3mm_D2.5mm_P10.16mm_Horizontal
- R2: value 10k -> 1k; footprint Resistor_SMD:R_0805_2012Metric -> Resistor_THT:R_Axial_DIN0207_L6.3mm_D2.5mm_P10.16mm_Horizontal
- R22: value 10k -> 0.01; footprint Resistor_SMD:R_0805_2012Metric -> Resistor_THT:R_Axial_DIN0411_L9.9mm_D3.6mm_P15.24mm_Horizontal
- R25: value 4k7 -> 10k; footprint Resistor_SMD:R_0805_2012Metric -> Resistor_THT:R_Axial_DIN0207_L6.3mm_D2.5mm_P10.16mm_Horizontal
- R26: value 2k2 -> 10k; footprint Resistor_SMD:R_0805_2012Metric -> Resistor_THT:R_Axial_DIN0207_L6.3mm_D2.5mm_P10.16mm_Horizontal
- R27: value 2k2 -> 1k; footprint Resistor_SMD:R_0805_2012Metric -> Resistor_THT:R_Axial_DIN0207_L6.3mm_D2.5mm_P10.16mm_Horizontal
- R29, R8: value 100k -> 1k; footprint Resistor_SMD:R_0805_2012Metric -> Resistor_THT:R_Axial_DIN0207_L6.3mm_D2.5mm_P10.16mm_Horizontal
- R4: value 2k -> 10k; footprint Resistor_SMD:R_0805_2012Metric -> Resistor_THT:R_Axial_DIN0207_L6.3mm_D2.5mm_P10.16mm_Horizontal
- R6: value 30k -> 1k; footprint Resistor_SMD:R_0805_2012Metric -> Resistor_THT:R_Axial_DIN0207_L6.3mm_D2.5mm_P10.16mm_Horizontal
Connections:
- net EC_ADC is gone; now on an unnamed net: R18.2
- net INA_INP is gone; now on an unnamed net: C3.1
- net PH_ADC is gone; now on an unnamed net: R17.2
- net at R16.2: now also R13.2; no longer JP1.1 (A)
- net at R17.1: now also R11.1, R14.1, U11.1 (Pin_1), U12.1 (Pin_1), U13.1 (Pin_1)
- net at R2.1: now also U5.3; no longer R1.2
- net at R3.2: now also Q1.3 (D), Q2.1 (G)
- net at J10.1 (Pin_1): now also J6.2 (Pin_2), J4.2 (Pin_2), J7.2 (Pin_2), J8.2 (G), U2.2 (Pin_2), U2.4 (Pin_4)
- net at R5.2: now also U6.6 (SCL)
- net at C3.2: now also JP1.2 (B), J_PI1.20 (Pin_20), J_PI1.30 (Pin_30), J_PI1.34 (Pin_34), J_PI1.6 (Pin_6), U6.2 (A1), U6.3 (A2), U6.4 (GND)
- net at R4.1: now also R5.1, J_PI1.14 (Pin_14), U6.8 (VCC)
- net at R19.2: now also R15.2, R21.2, R22.2, R24.2, D10.2 (A), D7.2 (A), D9.2 (A), Q9.3 (S), U19.5, U19.9
- net at J10.2 (Pin_2): now also R10.2, J_PI1.7 (Pin_7)
- net at J11.1 (Pin_1): now also D3.1 (K), D4.1 (K), J13.1 (Pin_1)
- net at R9.2: no longer R10.1
- net at C1.1: now also U1.2 (Pin_2), U10.1 (Pin_1), U4.13 (R), U8.1 (Pin_1), U9.7 (Pin_7)
- net at R23.2, R24.1: now also Q9.1 (G)
- net at R20.2, R21.1: now also Q8.1 (G)
- net at R18.1: now also Q7.1 (G)
- net at R28.2: now also D9.1 (K), U16.1 (Pin_1); no longer R29.1
- net +12V: no longer names the net of R3.1
- net +12V: now also D2.1 (K), D6.1 (K), J14.1 (Pin_1), J15.1 (Pin_1), Q2.3 (S), R_SHUNT1.1, U1.5 (Pin_5)
- net +12V_IN: no longer names the net of F1.1, J1.1 (Pin_1)
- removed net +3V3: C2.1, J6.1 (Pin_1), R15.2, R19.1, R22.1, R25.1, R26.1, R27.1
- net +3V3_PI: no longer names the net of R16.1
- net +3V3_PI: now also Q6.3 (S), U8.5 (Pin_5)
- net +5V_BAT: no longer names the net of R6.1
- net +5V_BAT: now also J_PI1.16 (Pin_16)
- net +5V_IN: no longer names the net of R1.1
- removed net +5V_MAINS: R13.1, R5.1, R9.1
- net 12V_FUSED: no longer names the net of F1.2
- net 12V_FUSED: now also D2.2 (A); no longer C1.2
- net BST_FB: no longer names the net of R6.2
- net BST_FB: now also R7.2, Q3.2 (G); no longer R7.1
- net BUZZ: no longer names the net of R28.1
- net BUZZ: now also R29.1
- net EC_EN: no longer names the net of R23.1
- net EC_EN: now also U15.1 (Pin_1)
- removed net GND: C2.2, J1.2 (Pin_2), J11.2 (Pin_2), J6.2 (Pin_2), JP1.2 (B), R10.2, R12.2, R14.2, R2.2, R21.2, R24.2, R29.2, R4.2, R7.2
- net GND_ISO: no longer names the net of J10.3 (Pin_3)
- net GND_ISO: now also R10.1
- net MAINS_N: no longer names the net of R15.1
- net MAINS_N: now also R14.2, Q6.1 (G)
- net PH_EN: no longer names the net of R20.1
- net PH_EN: now also U14.1 (Pin_1)
- net SCL: no longer names the net of J6.3 (Pin_3)
- net SCL: now also J3.3 (Pin_3), J5.3 (Pin_3), J_PI1.3 (Pin_3), U1.4 (Pin_4), U18.3 (Pin_3), U7.8 (Pin_8), U8.8 (Pin_8), U9.1 (Pin_1); no longer R27.2
- net SDA: no longer names the net of J6.4 (Pin_4)
- net SDA: now also J3.4 (Pin_4), J4.4 (Pin_4), J5.4 (Pin_4), U7.9 (Pin_9); no longer R26.2
- net VBAT_F: no longer names the net of R8.1
- net VBAT_F: no longer R11.1
- net VBAT_SENSE: no longer names the net of R11.2, R12.1
- net VBAT_SENSE: now also Q5.1 (G)
- net W1: no longer names the net of R25.2
- net W1: now also J_PI1.13 (Pin_13)
- new net: R4.2, U6.5 (SDA)
- new net: U4.6 (Q), U5.1
- new net: J_PI1.22 (Pin_22), U5.2
- new net: D6.2 (A), J14.2 (Pin_2), Q8.2 (D)
- new net: Q8.3 (S), R22.1, U9.3 (Pin_3)
- new net: R25.1, U18.1 (Pin_1), U4.16 (VDD), U4.3 (R), U5.14 (VDD)
- new net: U18.2 (Pin_2), U5.7 (VSS)
- new net: J3.2 (Pin_2), U7.1 (Pin_1), U7.6 (Pin_6), U8.2 (Pin_2)
- new net: J8.3 (S), U7.3 (Pin_3)
- new net: Q7.3 (S), R19.1, U7.5 (Pin_5)
- new net: U19.2, U19.3
- new net: J_PI1.11 (Pin_11), U19.4
- new net: D5.1 (K), Q2.2 (D)
- new net: Q10.1 (S), U19.11, U19.13, U19.7 (VSS)
- new net: C1.2, J_PI1.25 (Pin_25), J_PI1.9 (Pin_9), Q1.1 (S), U2.1 (Pin_1), U5.12, U5.13, U5.5, U5.8, U5.9
- new net: J7.1 (Pin_1), U2.3 (Pin_3)
- new net: R_SHUNT1.2, U1.6 (Pin_6)
- new net: U4.8 (VSS), U8.6 (Pin_6), U9.2 (Pin_2), U9.4 (Pin_4)
- new net: D8.1 (K), U20.1 (+), U3.1 (Pin_1)
- new net: D5.2 (A), J13.2 (Pin_2), Q7.2 (D)
- new net: J3.1 (Pin_1), J5.1 (Pin_1), J6.1 (Pin_1), Q4.1 (D), R9.1, U8.7 (Pin_7)
- new net: Q5.3 (S), R13.1, U8.3 (Pin_3)
- new net: J4.1 (Pin_1), Q3.1 (D), R26.1, R7.1, U3.3 (Pin_3)
- new net: D3.2 (A), J11.2 (Pin_2), Q5.2 (D)
- new net: J9.1 (V), Q4.3 (S)
- new net: J15.2 (Pin_2), Q9.2 (D)
- new net: J_PI1.15 (Pin_15), R27.1
- new net: Q10.2 (G), R27.2
- new net: D4.2 (A), J12.2 (Pin_2), Q6.2 (D)
- new net: D7.1 (K), R26.2
- new net: J2.1 (Pin_1), J_PI1.32 (Pin_32)
- new net: J2.2 (Pin_2), J_PI1.33 (Pin_33)
- new net: J16.2 (Pin_2), J5.2 (Pin_2), J9.2 (G), R12.2, U3.2 (Pin_2)
- new net: U10.3 (Pin_3), U9.9 (Pin_9)
- new net: J_PI1.1 (Pin_1), J_PI1.17 (Pin_17)
- new net: J7.4 (Pin_4), J_PI1.10 (Pin_10)
- new net: J_PI1.12 (Pin_12), U4.4 (Clk+)
- new net: J_PI1.39 (Pin_39), U6.1 (A0)
- new net: J_PI1.5 (Pin_5), U1.3 (Pin_3), U18.4 (Pin_4)
- new net: J7.3 (Pin_3), J_PI1.8 (Pin_8)
- new net: J8.1 (V), Q3.3 (S)
- new net: C2.1, R1.2, U4.2 (RxCx)
- new net: U1.1 (Pin_1), U4.5 (Clk-)
- new net: D8.2 (A), Q10.3 (D)
- new net: U10.2 (Pin_2), U4.11 (Clk-), U4.12 (Clk+)
- new net: R29.2, U17.1 (Pin_1)
- new net: C2.2, U4.1 (Cx)
- no-connect marks 20 -> 28
Other:
- note removed: "3.3 v for the sensors: AMS1117"
- note removed: "5 v for the pi: TPS565208, 5 a, into the header"
- note removed: "ads1115, the gravity probe boards, one probe powered at a time"
- note removed: "hat id eeprom: 24C32 on id_sd / id_sc"
- note removed: "isolated rs485 expansion: ADM2483, B0505S"
- note removed: "mounting holes"
- note removed: "oled, buzzer"
- note removed: "power in: 12 v brick, ideal diode, fuse, current monitor"
- note removed: "raspberry pi 4b header"
- note removed: "to the load board: 12 v out, heartbeat, fault"
- note removed: "ups: MCP73831 charger, 18650, XL6009 boost, two ideal diodes onto +5V"
- note removed: "water temp, air, light, co2, rtc"
- company: vertical hydroponic garden -> vertical gardening, no pico
- title: tower hat rev d -> garden hat, no pico (all through-hole)
