File: PCB/kicad/hat/hat.kicad_pcb (KiCad board)
At the start: 4 copper layers, 150 x 132 mm, 136 parts, among them J1 12V IN, J10 RS485 A B G, J11 12V OUT, J12 HB FLT GND, J2 spare gpio, J3 pH board, J4 EC board, J5 DS18B20, J6 sht31 module, J7 veml7700 module, J8 scd40 module, J9 oled ssd1306, Q1 AOD4184A, Q10 2N7002, Q2 2N7002, Q3 AOD4184A, Q4 AOD4184A, Q5 2N7002, Q6 AO3401A, Q7 2N7002, Q8 AO3401A, Q9 2N7002, U1 LM74700-Q1, U10 ADS1115 module, U11 DS3231MZ, U12 ADM2483BRWZ, U13 B0505S-1WR3, U2 INA226, U3 TPS565208, U4 MCP73831T-2ACI, U5 XL6009E1, U6 LM74700-Q1, U7 LM74700-Q1, U8 AMS1117-3.3, U9 24LC32A

Commit message: i redid everything for one board, one pi 5, and cut some features
Parts:
- removed BT1: 18650 protected, Battery:BatteryHolder_Keystone_1042_1x18650
- removed BT2: CR1220, Battery:BatteryHolder_Keystone_3000_1x12mm
- removed BZ1: active 5V, Buzzer_Beeper:Buzzer_12x9.5RM7.6
- removed C10, C14, C15, C20, C23, C8, C9: 22u 10V, Capacitor_SMD:C_1206_3216Metric
- removed C11, C21, C24, C25, C26, C28, C29, C32, C33, C34, C7: 100n, Capacitor_SMD:C_0805_2012Metric
- removed C12, C13, C35, C36: 4u7, Capacitor_SMD:C_0805_2012Metric
- removed C16: 220u 10V, Capacitor_THT:CP_Radial_D8.0mm_P3.50mm
- removed C17, C18: 1u, Capacitor_SMD:C_0805_2012Metric
- removed C19: 470u 10V, Capacitor_THT:CP_Radial_D8.0mm_P3.50mm
- removed C22, C27, C30, C31: 10u, Capacitor_SMD:C_1206_3216Metric
- removed C4: 470u 25V, Capacitor_THT:CP_Radial_D10.0mm_P5.00mm
- removed C5, C6: 10u 25V, Capacitor_SMD:C_1206_3216Metric
- removed F2, F3: 3A, Fuse:Fuse_1206_3216Metric
- removed F4: 7.5A blade, Fuse:FuseHolder_Blade_ATO_Littelfuse_FLR_178.6165
- removed H1, H2, H3, H4, H5, H6: M2.5, MountingHole:MountingHole_2.7mm_M2.5
- removed JP1: WP, Jumper:SolderJumper-2_P1.3mm_Open_Pad1.0x1.5mm
- removed JP2: term, Jumper:SolderJumper-2_P1.3mm_Open_Pad1.0x1.5mm
- removed the J_PI at (93.4, 4.77)
- removed L1: 4.7u 6A, Inductor_SMD:L_Bourns_SRP7028A_7.3x6.6mm
- removed L2: 22u 4A, Inductor_SMD:L_Bourns_SRP7028A_7.3x6.6mm
- removed R30: 120R, Resistor_SMD:R_0805_2012Metric
- removed R31, R32: 47k, Resistor_SMD:R_0805_2012Metric
- removed R33: 10k, Resistor_SMD:R_0805_2012Metric
- removed R34: 100R, Resistor_SMD:R_0805_2012Metric
- removed R_SENSE1, R_SENSE2: 10R, Resistor_SMD:R_0805_2012Metric
- removed the R_SHUNT at (87.9, 61.2)
- removed TP1: AIN3, TestPoint:TestPoint_Pad_D1.5mm
- added D10: pump, LED_D3.0mm, F.Cu at (137.2, 255.1)
- added J13: pump 3, TerminalBlock_CUI_TB007-508-02_1x02_P5.08mm_Horizontal, F.Cu at (134.3, 201.8)
- added J14: led strip, TerminalBlock_CUI_TB007-508-02_1x02_P5.08mm_Horizontal, F.Cu at (272.4, 201.8)
- added J15: fan, TerminalBlock_CUI_TB007-508-02_1x02_P5.08mm_Horizontal, F.Cu at (111.4, 230.0)
- added J16: flow sensor, TerminalBlock_CUI_TB007-508-03_1x03_P5.08mm_Horizontal, F.Cu at (220.7, 230.0)
- added J_PI: Pi 5, 40 pin (tall stacking header), PinSocket_2x20_P2.54mm_Vertical, F.Cu at (131.4, 59.0)
- added MTG1: MountingHole, MountingHole_2.7mm_M2.5, F.Cu at (178.4, 255.8)
- added MTG2: MountingHole, MountingHole_2.7mm_M2.5, F.Cu at (198.7, 255.8)
- added MTG3: MountingHole, MountingHole_2.7mm_M2.5, F.Cu at (219.0, 255.8)
- added MTG4: MountingHole, MountingHole_2.7mm_M2.5, F.Cu at (239.3, 255.8)
- added MTG5: MountingHole, MountingHole_2.7mm_M2.5, F.Cu at (259.6, 255.8)
- added MTG6: MountingHole, MountingHole_2.7mm_M2.5, F.Cu at (279.9, 255.8)
- added R_SHUNT: 5m, R_Axial_DIN0411_L9.9mm_D3.6mm_P15.24mm_Horizontal, F.Cu at (126.7, 18.8)
- added U14: PCA9685 ch3 (led pwm), PinHeader_1x01_P2.54mm_Vertical, F.Cu at (253.4, 91.0)
- added U15: PCA9685 ch4 (fan pwm), PinHeader_1x01_P2.54mm_Vertical, F.Cu at (282.3, 91.0)
- added U16: PCA9685 ch5 (rail status led), PinHeader_1x01_P2.54mm_Vertical, F.Cu at (26.7, 140.2)
- added U17: PCA9685 ch6 (pump status led), PinHeader_1x01_P2.54mm_Vertical, F.Cu at (60.9, 140.2)
- added U18: DS3231 RTC module, PinHeader_1x04_P2.54mm_Vertical, F.Cu at (86.5, 144.9)
- added U19: CD40106, DIP-14_W7.62mm, F.Cu at (289.8, 231.8)
- added U20: 5V active, Buzzer_12x9.5RM7.6, F.Cu at (55.8, 259.3)
- C1: value 1u 50V -> 100n; footprint Capacitor_SMD:C_0805_2012Metric -> C_Disc_D3.0mm_W2.0mm_P2.50mm
- C2: value 100n -> 10u 10V; footprint Capacitor_SMD:C_0805_2012Metric -> C_Disc_D3.0mm_W2.0mm_P2.50mm
- C3: footprint Capacitor_SMD:C_0805_2012Metric -> C_Disc_D3.0mm_W2.0mm_P2.50mm
- D1: value SMBJ15A -> 1.5KE15A; footprint Diode_SMD:D_SMB -> D_DO-201AE_P15.24mm_Horizontal
- D2: value charging -> SB5H100; footprint LED_SMD:LED_0805_2012Metric -> D_DO-201AD_P15.24mm_Horizontal
- D3: value SS34 -> 1N5819; footprint Diode_SMD:D_SMA -> D_DO-41_SOD81_P10.16mm_Horizontal
- D4, D5: value SMF5.0A -> 1N5819; footprint Diode_SMD:D_SOD-123F -> D_DO-41_SOD81_P10.16mm_Horizontal
- D6: value SMF5.0A -> 1N5822; footprint Diode_SMD:D_SOD-123F -> D_DO-201AD_P15.24mm_Horizontal
- D7: value SS14 -> 1N4148; footprint Diode_SMD:D_SMA -> D_DO-35_SOD27_P7.62mm_Horizontal
- D8: value SMAJ6.5CA -> 1N5819; footprint Diode_SMD:D_SMA -> D_DO-41_SOD81_P10.16mm_Horizontal
- D9: value SMAJ6.5CA -> rail; footprint Diode_SMD:D_SMA -> LED_D3.0mm
- F1: value 10A blade -> 10A; footprint Fuse:FuseHolder_Blade_ATO_Littelfuse_FLR_178.6165 -> FuseHolder_Blade_ATO_Littelfuse_FLR_178.6165
- J1: footprint TerminalBlock_CUI:TerminalBlock_CUI_TB007-508-02_1x02_P5.08mm_Horizontal -> TerminalBlock_CUI_TB007-508-02_1x02_P5.08mm_Horizontal
- J10: value RS485 A B G -> DS18B20; footprint TerminalBlock_CUI:TerminalBlock_CUI_TB007-508-03_1x03_P5.08mm_Horizontal -> TerminalBlock_CUI_TB007-508-03_1x03_P5.08mm_Horizontal
- J11: value 12V OUT -> pump 1; footprint TerminalBlock_CUI:TerminalBlock_CUI_TB007-508-02_1x02_P5.08mm_Horizontal -> TerminalBlock_CUI_TB007-508-02_1x02_P5.08mm_Horizontal
- J12: value HB FLT GND -> pump 2; footprint Connector_JST:JST_XH_B3B-XH-A_1x03_P2.50mm_Vertical -> TerminalBlock_CUI_TB007-508-02_1x02_P5.08mm_Horizontal
- J2: footprint Connector_PinHeader_2.54mm:PinHeader_1x04_P2.54mm_Vertical -> PinHeader_1x02_P2.54mm_Vertical
- J3: value pH board -> sht31 module; footprint revd:Gravity_TB3 -> PinHeader_1x04_P2.54mm_Vertical
- J4: value EC board -> veml7700 module; footprint revd:Gravity_TB3 -> PinHeader_1x04_P2.54mm_Vertical
- J5: value DS18B20 -> scd40 module; footprint TerminalBlock_CUI:TerminalBlock_CUI_TB007-508-03_1x03_P5.08mm_Horizontal -> PinHeader_1x04_P2.54mm_Vertical
- J6: value sht31 module -> oled ssd1306; footprint Connector_PinHeader_2.54mm:PinHeader_1x04_P2.54mm_Vertical -> PinHeader_1x04_P2.54mm_Vertical
- J7: value veml7700 module -> JSN-SR04T (uart mode); footprint Connector_PinHeader_2.54mm:PinHeader_1x04_P2.54mm_Vertical -> TerminalBlock_CUI_TB007-508-04_1x04_P5.08mm_Horizontal
- J8: value scd40 module -> pH board; footprint Connector_PinHeader_2.54mm:PinHeader_1x04_P2.54mm_Vertical -> Gravity_TB3
- J9: value oled ssd1306 -> EC board; footprint Connector_PinHeader_2.54mm:PinHeader_1x04_P2.54mm_Vertical -> Gravity_TB3
- Q1: value AOD4184A -> 2N7000; footprint Package_TO_SOT_SMD:TO-252-2 -> TO-92_Inline
- Q10: value 2N7002 -> 2N7000; footprint Package_TO_SOT_SMD:SOT-23 -> TO-92_Inline
- Q2: value 2N7002 -> IRF9540N; footprint Package_TO_SOT_SMD:SOT-23 -> TO-220-3_Vertical
- Q3, Q4: value AOD4184A -> BS250; footprint Package_TO_SOT_SMD:TO-252-2 -> TO-92_Inline
- Q5, Q7, Q9: value 2N7002 -> IRLZ44N; footprint Package_TO_SOT_SMD:SOT-23 -> TO-220-3_Vertical
- Q6, Q8: value AO3401A -> IRLZ44N; footprint Package_TO_SOT_SMD:SOT-23 -> TO-220-3_Vertical
- R1: value 56k2 -> 470k; footprint Resistor_SMD:R_0805_2012Metric -> R_Axial_DIN0207_L6.3mm_D2.5mm_P10.16mm_Horizontal
- R10: value 100k -> 4k7; footprint Resistor_SMD:R_0805_2012Metric -> R_Axial_DIN0207_L6.3mm_D2.5mm_P10.16mm_Horizontal
- R11, R14: value 100k -> 100R; footprint Resistor_SMD:R_0805_2012Metric -> R_Axial_DIN0207_L6.3mm_D2.5mm_P10.16mm_Horizontal
- R12, R21, R24, R3, R9: value 100k -> 10k; footprint Resistor_SMD:R_0805_2012Metric -> R_Axial_DIN0207_L6.3mm_D2.5mm_P10.16mm_Horizontal
- R13: value 100k -> 0.1; footprint Resistor_SMD:R_0805_2012Metric -> R_Axial_DIN0411_L9.9mm_D3.6mm_P15.24mm_Horizontal
- R15, R28, R7: footprint Resistor_SMD:R_0805_2012Metric -> R_Axial_DIN0207_L6.3mm_D2.5mm_P10.16mm_Horizontal
- R16, R19: value 10k -> 0.1; footprint Resistor_SMD:R_0805_2012Metric -> R_Axial_DIN0411_L9.9mm_D3.6mm_P15.24mm_Horizontal
- R17, R20, R23: value 1k -> 100R; footprint Resistor_SMD:R_0805_2012Metric -> R_Axial_DIN0207_L6.3mm_D2.5mm_P10.16mm_Horizontal
- R18, R5: value 1k -> 10k; footprint Resistor_SMD:R_0805_2012Metric -> R_Axial_DIN0207_L6.3mm_D2.5mm_P10.16mm_Horizontal
- R2: value 10k -> 1k; footprint Resistor_SMD:R_0805_2012Metric -> R_Axial_DIN0207_L6.3mm_D2.5mm_P10.16mm_Horizontal
- R22: value 10k -> 0.01; footprint Resistor_SMD:R_0805_2012Metric -> R_Axial_DIN0411_L9.9mm_D3.6mm_P15.24mm_Horizontal
- R25: value 4k7 -> 10k; footprint Resistor_SMD:R_0805_2012Metric -> R_Axial_DIN0207_L6.3mm_D2.5mm_P10.16mm_Horizontal
- R26: value 2k2 -> 10k; footprint Resistor_SMD:R_0805_2012Metric -> R_Axial_DIN0207_L6.3mm_D2.5mm_P10.16mm_Horizontal
- R27: value 2k2 -> 1k; footprint Resistor_SMD:R_0805_2012Metric -> R_Axial_DIN0207_L6.3mm_D2.5mm_P10.16mm_Horizontal
- R29, R8: value 100k -> 1k; footprint Resistor_SMD:R_0805_2012Metric -> R_Axial_DIN0207_L6.3mm_D2.5mm_P10.16mm_Horizontal
- R4: value 2k -> 10k; footprint Resistor_SMD:R_0805_2012Metric -> R_Axial_DIN0207_L6.3mm_D2.5mm_P10.16mm_Horizontal
- R6: value 30k -> 1k; footprint Resistor_SMD:R_0805_2012Metric -> R_Axial_DIN0207_L6.3mm_D2.5mm_P10.16mm_Horizontal
- U1: value LM74700-Q1 -> INA226 module 0x40; footprint Package_TO_SOT_SMD:SOT-23-6 -> PinHeader_1x06_P2.54mm_Vertical
- U10: value ADS1115 module -> PCA9685 module (i2c); footprint revd:ADS1115_Module -> PinHeader_1x04_P2.54mm_Vertical
- U11: value DS3231MZ -> PCA9685 ch0 (pump1 pwm); footprint Package_SO:SOIC-8_3.9x4.9mm_P1.27mm -> PinHeader_1x01_P2.54mm_Vertical
- U12: value ADM2483BRWZ -> PCA9685 ch1 (pump2 pwm); footprint Package_SO:SOIC-16W_7.5x10.3mm_P1.27mm -> PinHeader_1x01_P2.54mm_Vertical
- U13: value B0505S-1WR3 -> PCA9685 ch2 (pump3 pwm); footprint revd:B0505S_SIP4 -> PinHeader_1x01_P2.54mm_Vertical
- U2: value INA226 -> buck module 12V->5V; footprint Package_SO:MSOP-10_3x3mm_P0.5mm -> PinHeader_1x04_P2.54mm_Vertical
- U3: value TPS565208 -> AMS1117 3.3V module; footprint Package_TO_SOT_SMD:SOT-23-6 -> PinHeader_1x03_P2.54mm_Vertical
- U4: value MCP73831T-2ACI -> CD4538; footprint Package_TO_SOT_SMD:SOT-23-5 -> DIP-16_W7.62mm
- U5: value XL6009E1 -> CD4081; footprint revd:TO-263-5_TabNC -> DIP-14_W7.62mm
- U6: value LM74700-Q1 -> 24LC32A/P; footprint Package_TO_SOT_SMD:SOT-23-6 -> DIP-8_W7.62mm
- U7: value LM74700-Q1 -> ADS1115 module 0x48 (ph/ec + pump3 diff); footprint Package_TO_SOT_SMD:SOT-23-6 -> PinHeader_1x09_P2.54mm_Vertical
- U8: value AMS1117-3.3 -> ADS1115 module 0x49 (pump1/pump2 diff); footprint Package_TO_SOT_SMD:SOT-223-3_TabPin2 -> PinHeader_1x09_P2.54mm_Vertical
- U9: value 24LC32A -> ADS1115 module 0x4A (led diff); footprint Package_SO:SOIC-8_3.9x4.9mm_P1.27mm -> PinHeader_1x09_P2.54mm_Vertical
- moved D6 267.4 mm to (293.0, 199.5)
- moved R26 267.3 mm to (265.4, 226.3)
- moved R19 247.9 mm to (242.6, 198.7)
- moved R27 235.3 mm to (16.1, 254.5)
- moved R18 234.3 mm to (219.9, 198.1)
- moved R25 233.2 mm to (196.4, 226.3)
- moved Q7 229.6 mm to (178.7, 199.8)
- moved R17 223.1 mm to (197.6, 198.1)
- moved J8 221.2 mm to (238.7, 143.9)
- moved D7 215.0 mm to (245.6, 226.1)
- moved Q9 213.6 mm to (132.9, 228.0)
- moved Q10 211.1 mm to (39.1, 255.7)
- moved C2 210.3 mm to (301.3, 18.1)
- moved J11 205.5 mm to (154.3, 173.6), turned to 0 degrees
- moved R28 201.7 mm to (114.8, 254.5)
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Connections:
- net +12V_IN renamed +12V_RAW
- net Net-(Q9-G) renamed /FAN_G
- C1 pad 1: Net-(U1-VCAP) -> +3V3
- C1 pad 2: 12V_FUSED -> GND
- C2 pad 1: +3V3 -> MONO_RC
- C2 pad 2: GND -> MONO_CEXT
- C3 pad 1: /INA_INP -> +3V3_PI
- C3 pad 2: Net-(U2-Vin-) -> GND
- D1 pad 1: 12V_FUSED -> 12V_F
- D2 pad 1: Net-(D2-K) -> +12V
- D2 pad 2: Net-(D2-A) -> 12V_F
- D3 pad 1: +5V_BAT -> +12V_DOSE
- D3 pad 2: Net-(D3-A) -> /PUMP1_N
- D4 pad 1: /SDA -> +12V_DOSE
- D4 pad 2: GND -> /PUMP2_N
- D5 pad 1: /SCL -> +12V_DOSE
- D5 pad 2: GND -> /PUMP3_N
- D6 pad 1: /W1 -> +12V
- D6 pad 2: GND -> /LED_N
- D7 pad 1: +5V -> /FLOW_RAW
- D7 pad 2: Net-(BZ1--) -> GND
- D8 pad 1: Net-(D8-A1) -> +5V
- D8 pad 2: GND_ISO -> BUZZ_N
- D9 pad 1: Net-(D9-A1) -> /LED_STAT_RAIL
- D9 pad 2: GND_ISO -> GND
- F1 pad 2: 12V_FUSED -> 12V_F
- J10 pad 1: Net-(D8-A1) -> GND
- J10 pad 2: Net-(D9-A1) -> /W1
- J10 pad 3: GND_ISO -> +3V3
- J11 pad 1: Net-(J11-Pin_1) -> +12V_DOSE
- J11 pad 2: GND -> /PUMP1_N
- J12 pad 1: Net-(J12-Pin_1) -> +12V_DOSE
- J12 pad 2: /FLT -> /PUMP2_N
- J2 pad 1: Net-(J2-Pin_1) -> /SPARE_GPIO12
- J2 pad 2: Net-(J2-Pin_2) -> /SPARE_GPIO13
- J3 pad 1: PH_VCC -> +3V3
- J3 pad 3: Net-(J3-S) -> /SDA
- J4 pad 1: EC_VCC -> +3V3
- J4 pad 3: Net-(J4-S) -> /SDA
- J5 pad 3: /W1 -> /SDA
- J6 pad 3: /SCL -> /SDA
- J6 pad 4: /SDA -> /SCL
- J7 pad 1: +3V3 -> +5V
- J7 pad 3: /SCL -> /SONAR_TX
- J7 pad 4: /SDA -> /SONAR_RX
- J8 pad 1: +3V3 -> /PH_VCC_SW
- J8 pad 3: /SCL -> /PH_S
- J9 pad 1: GND -> /EC_VCC_SW
- J9 pad 2: +3V3 -> GND
- J9 pad 3: /SCL -> /EC_S
- Q1 pad 1: /ID_GATE -> GND
- Q1 pad 2: /12V_DIODE -> /RAIL_EN_R
- Q1 pad 3: 12V_FUSED -> /RAIL_G
- Q10 pad 1: Net-(Q10-G) -> GND
- Q10 pad 2: GND -> BUZZ_G
- Q10 pad 3: Net-(BZ1--) -> BUZZ_N
- Q2 pad 1: Net-(Q2-G) -> /RAIL_G
- Q2 pad 2: GND -> +12V_DOSE
- Q2 pad 3: Net-(Q2-D) -> +12V
- Q3 pad 1: Net-(Q3-G) -> +3V3
- Q3 pad 2: +5V -> PH_G
- Q3 pad 3: +5V_MAINS -> /PH_VCC_SW
- Q4 pad 1: Net-(Q4-G) -> +3V3
- Q4 pad 2: +5V -> EC_G
- Q4 pad 3: +5V_BAT -> /EC_VCC_SW
- Q5 pad 1: Net-(Q5-G) -> /PUMP1_G
- Q5 pad 2: GND -> /PUMP1_N
- Q5 pad 3: /MAINS_N -> /PUMP1_S
- Q6 pad 1: Net-(Q6-G) -> /PUMP2_G
- Q6 pad 2: +3V3 -> /PUMP2_N
- Q6 pad 3: PH_VCC -> /PUMP2_S
- Q7 pad 1: Net-(Q7-G) -> /PUMP3_G
- Q7 pad 2: GND -> /PUMP3_N
- Q7 pad 3: Net-(Q6-G) -> /PUMP3_S
- Q8 pad 1: Net-(Q8-G) -> /LED_G
- Q8 pad 2: +3V3 -> /LED_N
- Q8 pad 3: EC_VCC -> /LED_S
- Q9 pad 2: GND -> /FAN_N
- Q9 pad 3: Net-(Q8-G) -> GND
- R1 pad 1: +5V_IN -> +3V3
- R1 pad 2: Net-(U3-VFB) -> MONO_RC
- R10 pad 1: Net-(Q2-G) -> +3V3
- R10 pad 2: GND -> /W1
- R11 pad 1: VBAT_F -> /PUMP1_PWM
- R11 pad 2: /VBAT_SENSE -> /PUMP1_G
- R12 pad 1: /VBAT_SENSE -> /PUMP1_G
- R13 pad 1: +5V_MAINS -> /PUMP1_S
- R13 pad 2: Net-(Q5-G) -> GND
- R14 pad 1: Net-(Q5-G) -> /PUMP2_PWM
- R14 pad 2: GND -> /PUMP2_G
- R15 pad 1: /MAINS_N -> /PUMP2_G
- R15 pad 2: +3V3 -> GND
- R16 pad 1: +3V3_PI -> /PUMP2_S
- R16 pad 2: Net-(JP1-A) -> GND
- R17 pad 1: Net-(J3-S) -> /PUMP3_PWM
- R17 pad 2: /PH_ADC -> /PUMP3_G
- R18 pad 1: Net-(J4-S) -> /PUMP3_G
- R18 pad 2: /EC_ADC -> GND
- R19 pad 1: +3V3 -> /PUMP3_S
- R19 pad 2: Net-(Q6-G) -> GND
- R2 pad 1: Net-(U3-VFB) -> /RAIL_EN
- R2 pad 2: GND -> /RAIL_EN_R
- R20 pad 1: /PH_EN -> /LED_PWM
- R20 pad 2: Net-(Q7-G) -> /LED_G
- R21 pad 1: Net-(Q7-G) -> /LED_G
- R22 pad 1: +3V3 -> /LED_S
- R22 pad 2: Net-(Q8-G) -> GND
- R23 pad 1: /EC_EN -> /FAN_PWM
- R25 pad 2: /W1 -> /FAN_TACH
- R26 pad 2: /SDA -> /FLOW_RAW
- R27 pad 1: +3V3 -> /BUZZ
- R27 pad 2: /SCL -> BUZZ_G
- R28 pad 1: /BUZZ -> +3V3
- R28 pad 2: Net-(Q10-G) -> /LED_STAT_RAIL
- R29 pad 1: Net-(Q10-G) -> +3V3
- R29 pad 2: GND -> /LED_STAT_PUMP
- R3 pad 2: Net-(U3-EN) -> /RAIL_G
- R4 pad 1: Net-(U4-PROG) -> +3V3_PI
- R4 pad 2: GND -> /EEPROM_SDA
- R5 pad 1: +5V_MAINS -> +3V3_PI
- R5 pad 2: Net-(D2-A) -> /EEPROM_SCL
- R6 pad 1: +5V_BAT -> /PH_EN
- R6 pad 2: /BST_FB -> PH_G
- R7 pad 1: /BST_FB -> +3V3
- R7 pad 2: GND -> PH_G
- R8 pad 1: VBAT_F -> /EC_EN
- R8 pad 2: Net-(Q2-D) -> EC_G
- R9 pad 1: +5V_MAINS -> +3V3
- R9 pad 2: Net-(Q2-G) -> EC_G
- U1 pad 1: Net-(U1-VCAP) -> GND
- U1 pad 2: GND -> +3V3
- U1 pad 3: 12V_FUSED -> /SCL
- U1 pad 4: /12V_DIODE -> /SDA
- U1 pad 5: /ID_GATE -> +12V
- U1 pad 6: 12V_FUSED -> +12V_S
- U10 pad 1: GND -> +3V3
- U10 pad 2: unconnected-(U10-ALERT/RDY-Pad2) -> GND
- U10 pad 3: GND -> /SCL
- U10 pad 4: /PH_ADC -> /SDA
- U11 pad 1: unconnected-(U11-32KHZ-Pad1) -> /PUMP1_PWM
- U12 pad 1: +3V3 -> /PUMP2_PWM
- U13 pad 1: GND -> /PUMP3_PWM
- U2 pad 1: GND -> +12V_S
- U2 pad 3: unconnected-(U2-~{Alert}-Pad3) -> +5V
- U2 pad 4: /SDA -> GND
- U3 pad 1: GND -> +5V
- U3 pad 2: Net-(U3-SW) -> GND
- U3 pad 3: +12V -> +3V3
- U4 pad 1: Net-(D2-K) -> MONO_CEXT
- U4 pad 2: GND -> MONO_RC
- U4 pad 3: VBAT -> +3V3
- U4 pad 4: +5V_MAINS -> /HB_ALIVE
- U4 pad 5: Net-(U4-PROG) -> GND
- U5 pad 1: GND -> MONO_Q
- U5 pad 2: Net-(Q2-D) -> /ARM
- U5 pad 3: Net-(D3-A) -> /RAIL_EN
- U5 pad 4: VBAT_F -> (no net)
- U5 pad 5: /BST_FB -> GND
- U6 pad 1: Net-(U6-VCAP) -> GND
- U6 pad 3: +5V_MAINS -> GND
- U6 pad 4: +5V -> GND
- U6 pad 5: Net-(Q3-G) -> /EEPROM_SDA
- U6 pad 6: +5V_MAINS -> /EEPROM_SCL
- U7 pad 1: Net-(U7-VCAP) -> GND
- U7 pad 3: +5V_BAT -> /PH_S
- U7 pad 4: +5V -> /EC_S
- U7 pad 5: Net-(Q4-G) -> /PUMP3_S
- U7 pad 6: +5V_BAT -> GND
- U8 pad 1: GND -> +3V3
- U8 pad 2: +3V3 -> GND
- U8 pad 3: +5V -> /PUMP1_S
- U9 pad 1: GND -> /SDA
- U9 pad 3: GND -> /LED_S
- U9 pad 5: Net-(J_PI-Pin_27) -> (no net)
- U9 pad 6: Net-(J_PI-Pin_28) -> (no net)
- U9 pad 7: Net-(JP1-A) -> +3V3
- U9 pad 8: +3V3_PI -> /SDA
Routing:
- net /BUZZ: track 59.7 -> 699.6 mm, vias 1 -> 0
- net /LED_PWM: track 0.00 -> 584.7 mm, vias 0 -> 1
- net +12V_DOSE: track 0.00 -> 561.4 mm, vias 0 -> 10
- net /SDA: track 197.3 -> 732.4 mm, vias 6 -> 25
- net /SCL: track 188.5 -> 676.1 mm, vias 6 -> 15
- net +12V: track 245.0 -> 658.7 mm, vias 5 -> 10
- net /FLOW: track 0.00 -> 377.7 mm, vias 0 -> 1
- net /LED_N: track 0.00 -> 375.1 mm, vias 0 -> 2
- net /PUMP2_N: track 0.00 -> 355.1 mm, vias 0 -> 6
- net /PUMP3_S: track 0.00 -> 327.0 mm, vias 0 -> 4
- net GND: track 420.8 -> 107.5 mm, vias 68 -> 0
- net /PUMP1_S: track 0.00 -> 292.1 mm, vias 0 -> 4
- net MONO_Q: track 0.00 -> 292.0 mm
- net /PH_S: track 0.00 -> 281.3 mm, vias 0 -> 2
- net /FAN_PWM: track 0.00 -> 281.2 mm
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- added copper zone on In2.Cu, net +3V3
Other:
- board size 150 x 132 mm -> 330 x 282.6 mm

Commit message: pcb: shrunk board by about 47.5%
Parts:
- moved MTG1 298.6 mm to (9.50, 9.50)
- moved MTG5 286.9 mm to (9.50, 115.2)
- moved J12 277.5 mm to (16.4, 144.7)
- moved MTG2 246.7 mm to (213.4, 9.50)
- moved C2 236.6 mm to (79.3, 99.8)
- moved MTG4 232.4 mm to (9.50, 220.9)
- moved J16 224.2 mm to (23.4, 123.5)
- moved R26 223.4 mm to (63.3, 131.2)
- moved U15 220.7 mm to (79.2, 177.4)
- moved J9 211.5 mm to (196.6, 60.2)
- moved R13 204.6 mm to (59.5, 145.7)
- moved U19 201.3 mm to (106.8, 147.9)
- moved J1 199.2 mm to (208.2, 81.3)
- moved R7 197.6 mm to (122.9, 55.7)
- moved J7 194.7 mm to (22.0, 82.3)
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Routing:
- net /LED_PWM: track 584.7 -> 13.7 mm, vias 1 -> 0
- net /BUZZ: track 699.6 -> 230.6 mm, vias 0 -> 2
- net +12V_DOSE: track 561.4 -> 164.5 mm, vias 10 -> 0
- net +5V: track 525.7 -> 197.5 mm, vias 9 -> 0
- net MONO_RC: track 86.3 -> 391.3 mm, vias 2 -> 0
- net /PUMP2_N: track 355.1 -> 58.9 mm, vias 6 -> 0
- net +3V3: track 286.6 -> 0.00 mm, vias 1 -> 0
- net /FAN_PWM: track 281.2 -> 31.2 mm
- net MONO_Q: track 292.0 -> 46.3 mm
- net /PUMP2_PWM: track 261.1 -> 23.4 mm, vias 6 -> 0
- net /SDA: track 732.4 -> 504.9 mm, vias 25 -> 0
- net /PH_S: track 281.3 -> 56.0 mm, vias 2 -> 0
- net /LED_STAT_PUMP: track 248.2 -> 36.5 mm, vias 2 -> 0
- net /SCL: track 676.1 -> 471.2 mm, vias 15 -> 0
- net /PUMP3_S: track 327.0 -> 131.0 mm, vias 4 -> 0
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Other:
- board size 330 x 282.6 mm -> 216.8 x 226.3 mm
